File: Dragon32Issue2ASecam.kicad_pcb (KiCad board)
At the start: 2 copper layers, 253 x 199.1 mm, 59 parts, among them IC1 M3732H-20RS, IC15 MC6883, IC16 74LS244N, IC17 68A364, IC18 68A364, IC19 MC6809E, IC2 M3732H-20RS, IC3 M3732H-20RS, IC31 74LS02N, IC33 74LS138N, IC4 M3732H-20RS, IC5 M3732H-20RS, IC6 M3732H-20RS, IC7 M3732H-20RS, IC8 M3732H-20RS, SW1 RESET

Commit message: add PIA and VDG to schematics
Parts:
- added C26: 2.2nF, Capacitor_THT:C_Disc_D4.3mm_W1.9mm_P5.00mm, F.Cu at (107.2, 95.1)
- added C27: 0.1uF, Capacitor_THT:C_Disc_D4.3mm_W1.9mm_P5.00mm, F.Cu at (111.6, 99.7)
- added C30: 22nF, Capacitor_THT:C_Disc_D5.0mm_W2.5mm_P5.00mm, F.Cu at (117.2, 149.6)
- added C31: 22nF, Capacitor_THT:C_Disc_D5.0mm_W2.5mm_P5.00mm, F.Cu at (117.2, 152.7)
- added C32: 22nF, Capacitor_THT:C_Disc_D5.0mm_W2.5mm_P5.00mm, F.Cu at (117.2, 143.5)
- added C33: 22nF, Capacitor_THT:C_Disc_D5.0mm_W2.5mm_P5.00mm, F.Cu at (117.2, 146.6)
- added C35: 10uF, Capacitor_THT:CP_Radial_D5.0mm_P2.50mm, F.Cu at (151.3, 114.2)
- added C36: 100uF, Capacitor_THT:CP_Radial_D6.3mm_P2.50mm, F.Cu at (188.5, 100.1)
- added C38: 0.01uF, Capacitor_THT:C_Disc_D4.3mm_W1.9mm_P5.00mm, F.Cu at (119.2, 99.7)
- added C39: 0.01uF, Capacitor_THT:C_Disc_D4.3mm_W1.9mm_P5.00mm, F.Cu at (115.2, 67.6)
- added C42: 10uF, Capacitor_THT:CP_Radial_D5.0mm_P2.50mm, F.Cu at (161.5, 224.2)
- added C43: 0.01uF, Capacitor_THT:C_Disc_D4.3mm_W1.9mm_P5.00mm, F.Cu at (113.2, 165.9)
- added C44: 22nF, Capacitor_THT:C_Disc_D5.0mm_W2.5mm_P5.00mm, F.Cu at (118.1, 106.8)
- added C45: 0.01uF, Capacitor_THT:C_Disc_D4.3mm_W1.9mm_P5.00mm, F.Cu at (134.2, 223.4)
- added C48: 22pF, Capacitor_THT:C_Disc_D3.0mm_W2.0mm_P2.50mm, F.Cu at (141.4, 113.3)
- added D1: 1N914, Diode_THT:D_DO-35_SOD27_P12.70mm_Horizontal, F.Cu at (125.1, 77.3)
- added D2: 1N914, Diode_THT:D_DO-35_SOD27_P12.70mm_Horizontal, F.Cu at (109.7, 95.1)
- added D3: 1N914, Diode_THT:D_DO-35_SOD27_P12.70mm_Horizontal, F.Cu at (112.2, 82.4)
- added D7: 1N914, Diode_THT:D_DO-35_SOD27_P12.70mm_Horizontal, F.Cu at (110.4, 116.9)
- added D8: 1N914, Diode_THT:D_DO-35_SOD27_P12.70mm_Horizontal, F.Cu at (141.4, 129.4)
- added D9: 1N914, Diode_THT:D_DO-35_SOD27_P12.70mm_Horizontal, F.Cu at (154.1, 124.3)
- added IC12: MC6847, Package_DIP:DIP-40_W15.24mm, F.Cu at (177.9, 169.9)
- added IC13: 74LS273N, Package_DIP:DIP-20_W7.62mm, F.Cu at (238.4, 160.2)
- added IC20: MC14529B, Package_DIP:DIP-16_W7.62mm, F.Cu at (129.3, 140.1)
- added IC24: 74LS244N, Package_DIP:DIP-20_W7.62mm, F.Cu at (113.1, 170.6)
- added IC25: LM393P, Package_DIP:DIP-8_W7.62mm, F.Cu at (129.4, 121.9)
- added IC26: MC6821, Package_DIP:DIP-40_W15.24mm, F.Cu at (129.3, 169.8)
- added IC34: MC14050BCP, Package_DIP:DIP-16_W7.62mm, F.Cu at (160.0, 138.7)
- added IC35: MC6821, Package_DIP:DIP-40_W15.24mm, F.Cu at (152.8, 169.9)
- added L1: 3.3uH, Inductor_THT:L_Axial_L7.0mm_D3.3mm_P12.70mm_Horizontal_Fastron_MICC, F.Cu at (107.6, 71.1)
- added L2: 3.3uH, Inductor_THT:L_Axial_L7.0mm_D3.3mm_P12.70mm_Horizontal_Fastron_MICC, F.Cu at (111.6, 103.2)
- added PL1: Dragon Keyboard, Connector_PinHeader_2.54mm:PinHeader_1x16_P2.54mm_Vertical, F.Cu at (129.0, 240.8)
- added PL2: Printer, Connector_IDC:IDC-Header_2x10-1MP_P2.54mm_Latch_Horizontal, F.Cu at (98.9, 192.3)
- added PL3: DIN-6 J/S R, Dragon:DIN-6_DELTRON_671-0601_Horizontal, F.Cu at (98.8, 130.4)
- added PL4: DIN-5 (180) Cassette, Dragon:DIN-5_DELTRON_671-0501_45deg_Horizontal, F.Cu at (98.8, 110.3)
- added PL5: DIN-6 J/S L, Dragon:DIN-6_DELTRON_671-0601_Horizontal, F.Cu at (98.8, 90.3)
- added R16: 33K, Dragon:R_Axial_DIN0309_L9.0mm_D2.5mm_P12.70mm_Horizontal, F.Cu at (141.4, 121.8)
- added R29: 68K, Dragon:R_Axial_DIN0309_L9.0mm_D2.5mm_P12.70mm_Horizontal, F.Cu at (154.1, 119.2)
- added R30: 4K7, Dragon:R_Axial_DIN0309_L9.0mm_D2.5mm_P12.70mm_Horizontal, F.Cu at (141.4, 132.0)
- added R31: 4K7, Dragon:R_Axial_DIN0309_L9.0mm_D2.5mm_P12.70mm_Horizontal, F.Cu at (141.4, 126.8)
- added R32: 4K7, Dragon:R_Axial_DIN0309_L9.0mm_D2.5mm_P12.70mm_Horizontal, F.Cu at (112.4, 74.7)
- added R38: 4K7, Dragon:R_Axial_DIN0309_L9.0mm_D2.5mm_P12.70mm_Horizontal, F.Cu at (110.3, 156.1)
- added R42: 10K, Dragon:R_Axial_DIN0309_L9.0mm_D2.5mm_P12.70mm_Horizontal, F.Cu at (141.4, 155.4)
- added R43: 10K, Dragon:R_Axial_DIN0309_L9.0mm_D2.5mm_P12.70mm_Horizontal, F.Cu at (141.4, 158.0)
- added R45: 6K8, Dragon:R_Axial_DIN0309_L9.0mm_D2.5mm_P12.70mm_Horizontal, F.Cu at (110.4, 119.4)
- added R46: 220R, Dragon:R_Axial_DIN0309_L9.0mm_D2.5mm_P12.70mm_Horizontal, F.Cu at (110.4, 111.8)
- added R47: 8K2, Dragon:R_Axial_DIN0309_L9.0mm_D2.5mm_P12.70mm_Horizontal, F.Cu at (123.1, 114.3)
- added R48: 15K, Dragon:R_Axial_DIN0309_L9.0mm_D2.5mm_P12.70mm_Horizontal, F.Cu at (110.4, 132.1)
- added R49: 1K, Dragon:R_Axial_DIN0309_L9.0mm_D2.5mm_P12.70mm_Horizontal, F.Cu at (110.4, 121.9)
- added R50: 56K, Dragon:R_Axial_DIN0309_L9.0mm_D2.5mm_P12.70mm_Horizontal, F.Cu at (123.1, 127.0)
- added R51: 1M5, Dragon:R_Axial_DIN0309_L9.0mm_D2.5mm_P12.70mm_Horizontal, F.Cu at (123.1, 129.5)
- added R52: 56K, Dragon:R_Axial_DIN0309_L9.0mm_D2.5mm_P12.70mm_Horizontal, F.Cu at (123.1, 124.5)
- added R53: 10M, Dragon:R_Axial_DIN0309_L9.0mm_D2.5mm_P12.70mm_Horizontal, F.Cu at (110.4, 137.2)
- added R54: 1K, Dragon:R_Axial_DIN0309_L9.0mm_D2.5mm_P12.70mm_Horizontal, F.Cu at (110.4, 134.6)
- added R55: 10K, Dragon:R_Axial_DIN0309_L9.0mm_D2.5mm_P12.70mm_Horizontal, F.Cu at (110.4, 139.7)
- added R56: 10K, Dragon:R_Axial_DIN0309_L9.0mm_D2.5mm_P12.70mm_Horizontal, F.Cu at (141.4, 152.9)
- added R57: 20K 1%, Dragon:R_Axial_DIN0309_L9.0mm_D2.5mm_P12.70mm_Horizontal, F.Cu at (141.4, 137.0)
- added R58: 80K6 1%, Dragon:R_Axial_DIN0309_L9.0mm_D2.5mm_P12.70mm_Horizontal, F.Cu at (141.4, 147.2)
- added R59: 160K 1%, Dragon:R_Axial_DIN0309_L9.0mm_D2.5mm_P12.70mm_Horizontal, F.Cu at (141.4, 142.1)
- added R60: 330K 1%, Dragon:R_Axial_DIN0309_L9.0mm_D2.5mm_P12.70mm_Horizontal, F.Cu at (141.4, 139.6)
- added R61: 40K2 1%, Dragon:R_Axial_DIN0309_L9.0mm_D2.5mm_P12.70mm_Horizontal, F.Cu at (141.4, 144.7)
- added R62: 10K 1%, Dragon:R_Axial_DIN0309_L9.0mm_D2.5mm_P12.70mm_Horizontal, F.Cu at (141.4, 149.7)
- added R63: 4K7, Dragon:R_Axial_DIN0309_L9.0mm_D2.5mm_P12.70mm_Horizontal, F.Cu at (271.2, 98.5)
- added R64: 100K, Dragon:R_Axial_DIN0309_L9.0mm_D2.5mm_P12.70mm_Horizontal, F.Cu at (141.4, 134.5)
- added R72: 4K7, Dragon:R_Axial_DIN0309_L9.0mm_D2.5mm_P12.70mm_Horizontal, F.Cu at (141.4, 160.5)
- added RL1: OJS HM FORM A, Dragon:OJS HM 10A Relay, F.Cu at (120.2, 88.5)
- added TR1: BC141, Package_TO_SOT_THT:TO-92_Inline_Wide, F.Cu at (109.2, 79.3)
- C1: value 0.1uF -> 0.01uF
- R1: value 100K -> 100R
- moved C1 1.73 mm to (104.8, 67.6)
- moved R1 1.09 mm to (103.3, 64.8)
Connections:
- C1 pad 1: Net-(C1-Pad1) -> GND
- C1 pad 2: GND -> /PIA0/Joystick +V
- IC31 pad 4: (no net) -> STROBE
- IC31 pad 5: (no net) -> Net-(IC35-PA1)
- IC31 pad 6: (no net) -> Net-(IC35-PA1)
- R1 pad 1: Net-(C1-Pad1) -> +5V
- R1 pad 2: +5V -> /PIA0/Joystick +V
